Commit message: Add Nav2 sim harness, flat base_footprint frame, and Foxglove goal relay
Follow-up to the merged nav-stability fixes:

- go2_nav_sim: Tier-0 kinematic Nav2 test harness (accel-limited fake
  base, map raycast -> /scan, scenario scorecard). Runs the SAME
  nav2_params headless in Docker on macOS, viewed in Foxglove.
- base_footprint: driver publishes a yaw-only odom->base_footprint so the
  dog's body pitch/roll no longer tilts the 2D costmap or projected scan.
  All 2D consumers (Nav2, AMCL, slam_toolbox, pointcloud_to_laserscan)
  repointed to base_footprint; stale URDF base_footprint joints removed.
- goal_relay: bridge Foxglove's Publish tool (/goal_pose, /waypoint_add,
  /waypoints_run) into Nav2 NavigateToPose / FollowWaypoints; wired into
  navigation.launch.py and robot.launch.py (nav2:=true).
- scripts/: one-command run_mapping, run_mapping_nav, run_nav, save_map,
  run_sim, waypoint, and build_robot_image helpers.
- docker: reorder Dockerfile so pip/rosdep install from manifests before
  the source COPY (+ .dockerignore), so code edits no longer trigger the
  ~5-min dependency rebuild. Add sim service + entrypoint.
- gitignore /maps/ (local artifacts from save_map.sh).

Co-authored-by: Cursor <cursoragent@cursor.com>

File: go2_robot_sdk/urdf/go2.urdf (robot description, URDF)
Before this commit: robot go2, 33 links, 32 joints
Links:
- removed link base_footprint
Joints:
- removed joint base_footprint_joint

File: go2_robot_sdk/urdf/go2_with_realsense.urdf (robot description, URDF)
Before this commit: robot go2, 35 links, 34 joints
Links:
- removed link base_footprint
Joints:
- removed joint base_footprint_joint
